File: Adafruit CC3000 Breakout.brd (EAGLE design)
At the start: 39.4 x 59.7 mm, 34 parts, among them IC1 ATmega1284P, U1 CC3000MOD, X1 2500AT44M0400E

Commit message: Put CC3000 I2C pins on 0.1" pins.
Instead of test points.
Parts:
- removed TP1: SCL, microbuilder:TESTPOINT_PAD_1MM
- removed TP2: SDA, microbuilder:TESTPOINT_PAD_1MM
- added JP6: (no value), pinhead:1X02
- moved R2 4.91 mm to (27.3, 47.0)
Connections:
- net SCL_3V: now also JP6.1; no longer TP1.P$1
- net SDA_3V: now also JP6.2; no longer TP2.P$1
Routing:
- net SCL_3V: track 7.72 -> 3.27 mm, vias 1 -> 0
- net VBAT_EN_3V: track 4.39 -> 0.00 mm
- net SDA_3V: track 10.7 -> 6.66 mm, vias 1 -> 0
Changed lines of the file:
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@@
 </element>
 <element name="C8" library="rcl" package="C1206" value="10µF" x="31.75" y="39.37" rot="R90"/>
-<element name="TP1" library="microbuilder" package="TESTPOINT_PAD_1MM" value="SCL" x="16.5" y="43.77" smashed="yes" rot="MR0">
-<attribute name="NAME" x="15.557" y="43.343" size="0.8128" layer="26" ratio="18" rot="MR0"/>
-<attribute name="VALUE" x="17.599" y="42.945" size="1.016" layer="22" ratio="10" rot="MR90"/>
-</element>
-<element name="TP2" library="microbuilder" package="TESTPOINT_PAD_1MM" value="SDA" x="16.5" y="41.27" smashed="yes" rot="MR0">
-<attribute name="NAME" x="15.557" y="40.843" size="0.8128" layer="26" ratio="18" rot="MR0"/>
-<attribute name="VALUE" x="18.529" y="42.161" size="1.016" layer="22" ratio="10" rot="MR270"/>
-</element>
-<element name="R2" library="rcl" package="R1206" value="10K" x="22.4" y="47.27" smashed="yes" rot="R270">
-<attribute name="NAME" x="23.0875" y="45.4175" size="0.8128" layer="25" ratio="18" rot="R180"/>
-<attribute name="VALUE" x="18.859" y="49.1075" size="1.016" layer="27" font="vector" ratio="10" rot="R270"/>
+<element name="R2" library="rcl" package="R1206" value="10K" x="27.305" y="46.99" smashed="yes" rot="R270">
+<attribute name="NAME" x="27.9925" y="45.1375" size="0.8128" layer="25" ratio="18" rot="R180"/>
+<attribute name="VALUE" x="23.764" y="48.8275" size="1.016" layer="27" font="vector" ratio="10" rot="R270"/>
 </element>
 <element name="R3" library="rcl" package="R1206" value="10K" x="12.7" y="27.94" rot="R90"/>
@@
 <element name="JP3" library="pinhead" package="1X02" value="" x="36.83" y="19.05" rot="R270"/>
 <element name="JP4" library="pinhead" package="1X02" value="" x="36.83" y="13.97" rot="R90"/>
+<element name="JP6" library="pinhead" package="1X02" value="" x="23.495" y="46.99" rot="R270"/>
 </elements>
 <signals>
@@
 <wire x1="18.85" y1="48.02" x2="14.8" y2="48.02" width="0" layer="19" extent="1-1"/>
 <wire x1="20.7" y1="48.07" x2="18.85" y2="48.02" width="0" layer="19" extent="1-1"/>
-<wire x1="22.4" y1="48.692" x2="20.7" y2="48.07" width="0" layer="19" extent="1-1"/>
+<wire x1="27.305" y1="48.412" x2="20.7" y2="48.07" width="0" layer="19" extent="1-1"/>
 <wire x1="29.21" y1="40.77" x2="24.4" y2="41.67" width="0" layer="19" extent="1-1"/>
 <wire x1="31.75" y1="40.77" x2="29.21" y2="40.77" width="0" layer="19" extent="1-1"/>
@@
 <contactref element="U1" pad="30"/>
 <contactref element="U1" pad="29"/>
-<contactref element="TP1" pad="P$1"/>
 <wire x1="17.2" y1="48.02" x2="17.2" y2="48.97" width="0.25" layer="1"/>
 <wire x1="17.2" y1="48.97" x2="17" y2="49.17" width="0.25" layer="1"/>
 <wire x1="17" y1="49.17" x2="16.2" y2="49.17" width="0.25" layer="1"/>
+<wire x1="16.51" y1="49.17" x2="16.2" y2="49.17" width="0" layer="19" extent="1-16"/>
 <wire x1="16.2" y1="49.17" x2="16" y2="48.97" width="0.25" layer="1"/>
 <wire x1="16" y1="48.97" x2="16" y2="48.02" width="0.25" layer="1"/>
-<wire x1="16" y1="48.02" x2="16" y2="46.07" width="0.25" layer="1"/>
-<via x="16" y="46.07" extent="1-16" drill="0.4"/>
-<wire x1="16" y1="46.07" x2="16" y2="45.17" width="0.25" layer="16"/>
-<wire x1="16" y1="45.17" x2="16.5" y2="44.67" width="0.25" layer="16"/>
-<wire x1="16.5" y1="44.67" x2="16.5" y2="43.77" width="0.25" layer="16"/>
+<contactref element="JP6" pad="1"/>
+<wire x1="23.495" y1="48.26" x2="21.59" y2="50.8" width="0" layer="19" extent="1-16"/>
+<wire x1="21.59" y1="50.8" x2="17.78" y2="50.8" width="0" layer="19" extent="1-16"/>
+<wire x1="17.78" y1="50.8" x2="16.51" y2="49.53" width="0" layer="19" extent="1-16"/>
+<wire x1="16.51" y1="49.53" x2="16.51" y2="49.17" width="0" layer="19" extent="1-16"/>
 </signal>
 <signal name="SDA_3V">
 <contactref element="U1" pad="28"/>
 <contactref element="U1" pad="27"/>
-<contactref element="TP2" pad="P$1"/>
 <wire x1="18.85" y1="46.17" x2="19.7" y2="46.17" width="0.25" layer="1"/>
 <wire x1="19.7" y1="46.17" x2="19.9" y2="45.97" width="0.25" layer="1"/>
-<wire x1="19.9" y1="45.97" x2="19.9" y2="45.17" width="0.25" layer="1"/>
+<wire x1="19.9" y1="45.97" x2="19.9" y2="45.72" width="0.25" layer="1"/>
+<wire x1="19.9" y1="45.72" x2="19.9" y2="45.17" width="0.25" layer="1"/>
 <wire x1="19.9" y1="45.17" x2="19.7" y2="44.97" width="0.25" layer="1"/>
 <wire x1="19.7" y1="44.97" x2="18.85" y2="44.97" width="0.25" layer="1"/>
-<wire x1="16.5" y1="41.27" x2="17.5" y2="41.27" width="0.25" layer="16"/>
-<wire x1="17.5" y1="41.27" x2="17.7" y2="41.47" width="0.25" layer="16"/>
-<wire x1="17.7" y1="41.47" x2="17.7" y2="45.67" width="0.25" layer="16"/>
-<wire x1="17.7" y1="45.67" x2="17.3" y2="46.07" width="0.25" layer="16"/>
-<via x="17.3" y="46.07" extent="1-16" drill="0.4"/>
-<wire x1="18.85" y1="46.17" x2="17.4" y2="46.17" width="0.25" layer="1"/>
-<wire x1="17.4" y1="46.17" x2="17.3" y2="46.07" width="0.25" layer="1"/>
+<contactref element="JP6" pad="2"/>
+<wire x1="23.495" y1="45.72" x2="19.9" y2="45.72" width="0.254" layer="1"/>
 </signal>
 <signal name="VBAT" class="1">
@@
 <contactref element="R2" pad="2"/>
 <contactref element="IC1" pad="41"/>
-<wire x1="20.0152" y1="43.8404" x2="18.8976" y2="43.8404" width="0.2032" layer="1"/>
-<wire x1="21.9456" y1="45.7708" x2="20.0152" y2="43.8404" width="0.2032" layer="1"/>
-<wire x1="18.8976" y1="43.8404" x2="18.85" y2="43.77" width="0.2032" layer="1"/>
-<wire x1="21.9456" y1="45.7708" x2="22.4" y2="45.848" width="0.2032" layer="1"/>
+<wire x1="18.85" y1="43.77" x2="27.305" y2="45.568" width="0" layer="19" extent="1-1"/>
 <wire x1="16.18" y1="20.405" x2="18.85" y2="43.77" width="0" layer="19" extent="1-1"/>
 </signal>
